Commit message: Add Octmap

File: ss_description/urdf/quadrotor_with_camera.urdf.xacro (robot description, xacro)
@@ -25,4 +25,5 @@
     <gazebo>
       <plugin name="camera_controller" filename="libgazebo_ros_control.so">
+        <controlPeriod>0.01</controlPeriod>
         <robotSimType>gazebo_ros_control/DefaultRobotHWSim</robotSimType>
         <robotNamespace>$(arg robot_ns)/cam_control</robotNamespace>

File: ss_description/urdf/realsense.urdf.xacro (robot description, xacro)
@@ -94,4 +94,10 @@
       </collision>
     </link>
+    <joint name="${name}_depth_joint" type="fixed">
+      <origin xyz="0.0 0.0 0.0" rpy="0 0 0" />
+      <parent link="${name}_link" />
+      <child link="${name}_depth_frame"/>
+    </joint>
+    <link name="${name}_depth_frame"/>
     <gazebo reference="base_fixed_link">
       <material>Gazebo/Orange</material>
@@ -111,5 +117,5 @@
       </actuator>
     </transmission>
-    <gazebo reference="${name}_link">
+    <gazebo reference="${name}_depth_frame">
       <material>Gazebo/Grey</material>
       <sensor type="depth" name="${name}">
@@ -131,4 +137,5 @@
         <plugin name="${name}_camera_controller" filename="libgazebo_ros_openni_kinect.so">
           <cameraName>${name}</cameraName>
+          <bodyName>${name}_frame</bodyName>
           <imageTopicName>color/image_raw</imageTopicName>
           <cameraInfoTopicName>color/camera_info</cameraInfoTopicName>
@@ -136,5 +143,5 @@
           <depthImageCameraInfoTopicName>depth/camera_info</depthImageCameraInfoTopicName>
           <pointCloudTopicName>depth/points</pointCloudTopicName>
-          <frameName>${name}_color_optical_frame</frameName>
+          <frameName>${name}_depth_frame</frameName>
         </plugin>
       </sensor>
